File: elec/voyager_fc/voyager_fc.sch (KiCad schematic (older format))
At the start: 173 parts, among them J1 Raspberry Pi 5 Connector, J10 BM04B-GHS-TBT_LF__SN__N_, J11 BM04B-GHS-TBT_LF__SN__N_, J12 BM04B-GHS-TBT_LF__SN__N_, J13 BM04B-GHS-TBT_LF__SN__N_, J14 BM03B-GHS-TBT_LF__SN__N_, J15 BM03B-GHS-TBT_LF__SN__N_, J16 BM03B-GHS-TBT_LF__SN__N_, J17 BM03B-GHS-TBT_LF__SN__N_, J18 BM02B-GHS-TBT_LF__SN__N_, J19 BM02B-GHS-TBT_LF__SN__N_, J2 Pi Power Connect, J20 BM02B-GHS-TBT_LF__SN__N_, J21 BM06B-GHS-TBT_LF__SN__N_, J22 BM06B-GHS-TBT_LF__SN__N_, J23 BM06B-GHS-TBT_LF__SN__N_, J24 AUX Leak, J3 AUX Power Connect, J4 PWM Power Rail 1, J5 PWM GND Rail 1, J6 PWM Signal Rail 1, J7 PWM Power Rail 2, J8 PWM GND Rail 2, J9 PWM Signal Rail 2, Q3 BSS138, Q4 BSS138, Q5 MMBT3906, U1 TCA9548APWR, U10 LTC4311CDC_TRMPBF, U11 LTC4311CDC_TRMPBF, U12 LTC4311CDC_TRMPBF, U13 LTC4311CDC_TRMPBF, U14 TXS0102YZP, U15 TXS0102YZP, U16 TXS0102YZP, U17 TXS0102YZP, U2 PCA9685PW, U3 PCA9685PW, U4 BME680, U5 ICM-20948, U6 TPS2121RUXR, U7 AMS1117-3.3, U8 ADS1015IDGS, U9 AMS1117-1.8, X1 SG-8002CE

Commit message: Update voyager annotations
Parts:
- renumbered C7 to C1, C12 to C10, C19 to C11, C13 to C12, C20 to C13, C21 to C15, C15 to C16, C22 to C17, C16 to C18, C23 to C19, C8 to C2, C17 to C20, C10 to C21, C11 to C22, C53 to C23, C54 to C24, C24 to C25, C25 to C26, C26 to C27, C27 to C28, C31 to C29, C35 to C3, C28 to C30, C4 to C31, C29 to C32, C30 to C33, C36 to C34, C38 to C35, C40 to C36, C42 to C37, C37 to C38, C3 to C4, C41 to C40, C43 to C41, C32 to C42, C33 to C43, C0 to C44, C1 to C45, C51 to C46, C52 to C47, C49 to C48, C50 to C49, C44 to C50, C45 to C51, C46 to C52, C48 to C53, C9 to C54, C34 to C6, C2 to C7, C6 to C8, C18 to C9, D2 to D1, D3 to D2, D4 to D3, D1 to D4, J6 to J10, J14 to J11, J15 to J12, J16 to J13, J17 to J14, J2 to J15, J3 to J16, J10 to J17, J11 to J18, J12 to J19, J21 to J2, J13 to J20, J24 to J21, J18 to J22, J19 to J23, J20 to J24, J22 to J3, J23 to J4, J7 to J5, J8 to J6, J9 to J7, J4 to J8, J5 to J9, Q4 to Q1, Q3 to Q2, Q5 to Q3, R55 to R1, R17 to R10, R18 to R11, R19 to R12, R20 to R13, R21 to R14, R22 to R15, R23 to R16, R24 to R17, R25 to R18, R26 to R19, R56 to R2, R27 to R20, R58 to R21, R3 to R22, R28 to R23, R29 to R24, R30 to R25, R31 to R26, R32 to R27, R33 to R28, R34 to R29, R57 to R3, R35 to R30, R36 to R31, R37 to R32, R38 to R33, R39 to R34, R40 to R35, R41 to R36, R42 to R37, R43 to R38, R54 to R39, R2 to R4, R59 to R40, R62 to R41, R65 to R42, R68 to R43, R52 to R44, R53 to R45, R0 to R46, R50 to R48, R48 to R49, R12 to R5, R51 to R50, R49 to R51, R61 to R52, R60 to R53, R63 to R54, R64 to R55, R67 to R56, R66 to R57, R69 to R58, R70 to R59, R13 to R6, R71 to R60, R72 to R61, R73 to R62, R74 to R63, R8 to R64, R9 to R65, R10 to R66, R11 to R67, R45 to R68, R44 to R69, R14 to R7, R46 to R70, R15 to R8, R16 to R9, U4 to U1, U13 to U10, U7 to U11, U1 to U12, U14 to U13, U15 to U14, U16 to U15, U17 to U16, U5 to U17, U8 to U4, U6 to U5, U9 to U6, U10 to U7, U11 to U8, U12 to U9
Other:
- moved on the sheet: C34, C35, C36, C37, C38, C39, C40, C41, C46, C47, C48, C49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
