File: elec/voyager_fc/IMU.sch (KiCad schematic (older format))
At the start: 8 parts

Commit message: Place all components and start route
Parts:
- added C35: 10uF, Capacitor_SMD:C_0603_1608Metric, symbol Device:C_Small
- C36: renamed from C?; footprint Capacitor_SMD:C_0603_1608Metric -> Capacitor_SMD:C_0402_1005Metric
- gave numbers to parts that had none: 7
Connections:
- net +1V8: now also C35.2
- net GND: now also C35.1; no longer U7.21 (AUX_DA), U7.7 (AUX_CL)
- net SC2 renamed SCL
- net SCL21v8 renamed SCL21V8
- net SD2 renamed SDA
- net SDL21v8 renamed SDL21V8
- no-connect marks 0 -> 2
